Commit message: Decrease simulated velodyne min range and tune move_base parameters

File: bramblebee_description/urdf/velodyne_hdl32e.urdf.xacro (robot description, xacro)
@@ -2,5 +2,5 @@
 <robot xmlns:xacro="http://www.ros.org/wiki/xacro" name="Velodyne_HDL32E">
   <xacro:property name="M_PI" value="3.1415926535897931" />
-  <xacro:macro name="Velodyne_HDL32E" params="*origin parent:=base_link name:=velodyne topic:=/velodyne_points hz:=10 lasers:=32 samples:=2187 collision_range:=0.3 min_range:=0.9 max_range:=130.0 noise:=0.001 min_angle:=-${M_PI} max_angle:=${M_PI}">
+  <xacro:macro name="Velodyne_HDL32E" params="*origin parent:=base_link name:=velodyne topic:=/velodyne_points hz:=10 lasers:=32 samples:=2187 collision_range:=0.3 min_range:=0.1 max_range:=130.0 noise:=0.001 min_angle:=-${M_PI} max_angle:=${M_PI}"> <!-- min_range was 0.9 -->
     <joint name="${name}_base_mount_joint" type="fixed">
       <xacro:insert_block name="origin" />

Commit message: Fixed description with the lidar collision on the arm

File: bramblebee_description/urdf/velodyne_hdl32e.urdf.xacro (robot description, xacro)
@@ -2,5 +2,5 @@
 <robot xmlns:xacro="http://www.ros.org/wiki/xacro" name="Velodyne_HDL32E">
   <xacro:property name="M_PI" value="3.1415926535897931" />
-  <xacro:macro name="Velodyne_HDL32E" params="*origin parent:=base_link name:=velodyne topic:=/velodyne_points hz:=10 lasers:=32 samples:=2187 collision_range:=0.3 min_range:=0.1 max_range:=130.0 noise:=0.001 min_angle:=-${M_PI} max_angle:=${M_PI}"> <!-- min_range was 0.9 -->
+  <xacro:macro name="Velodyne_HDL32E" params="*origin parent:=base_link name:=velodyne topic:=/velodyne_points hz:=10 lasers:=32 samples:=2187 collision_range:=0.3 min_range:=0.9 max_range:=130.0 noise:=0.001 min_angle:=-${M_PI} max_angle:=${M_PI}"> <!-- min_range was 0.9 -->
     <joint name="${name}_base_mount_joint" type="fixed">
       <xacro:insert_block name="origin" />
