Commit message: Remove deprecated and unused parts from bramblebee description

File: bramblebee_description/urdf/bramblebee.urdf.xacro (robot description, xacro)
@@ -22,10 +22,4 @@
 -->
 <robot name="husky" xmlns:xacro="http://ros.org/wiki/xacro">
-  <xacro:arg name="laser_enabled" default="false" />
-  <xacro:arg name="laser_xyz" default="$(optenv HUSKY_LMS1XX_XYZ 0.2206 0.0 0.00635)" />
-  <xacro:arg name="laser_rpy" default="$(optenv HUSKY_LMS1XX_RPY 0.0 0.0 0.0)" />
-  <xacro:arg name="kinect_enabled" default="false" />
-  <xacro:arg name="kinect_xyz" default="$(optenv HUSKY_KINECT_XYZ 0 0 0)" />
-  <xacro:arg name="kinect_rpy" default="$(optenv HUSKY_KINECT_RPY 0 0.18 3.14)" />
   <xacro:arg name="robot_namespace" default="/" />
   <xacro:arg name="urdf_extras" default="empty.urdf" />
@@ -33,6 +27,4 @@
   <xacro:include filename="$(find husky_description)/urdf/decorations.urdf.xacro" />
   <xacro:include filename="$(find bramblebee_description)/urdf/bramblebee_wheel.urdf.xacro" />
-<!--   <xacro:include filename="$(find husky_description)/urdf/accessories/kinect_camera.urdf.xacro"/>
- -->  <xacro:include filename="$(find husky_description)/urdf/accessories/sick_lms1xx_mount.urdf.xacro"/>
   <xacro:include filename="$(find husky_description)/urdf/accessories/sensor_arch.urdf.xacro"/>
   <xacro:property name="M_PI" value="3.14159"/>
@@ -113,24 +105,4 @@
   </xacro:bramblebee_wheel>
   <xacro:husky_decorate />
-  <xacro:if value="$(arg laser_enabled)">
-    <sick_lms1xx_mount prefix="base"/>
-    <sick_lms1xx frame="base_laser" topic="scan" robot_namespace="$(arg robot_namespace)"/>
-    <joint name="laser_mount_joint" type="fixed">
-      <origin xyz="$(arg laser_xyz)" rpy="$(arg laser_rpy)" />
-      <parent link="top_plate_link" />
-      <child link="base_laser_mount" />
-    </joint>
-  </xacro:if>
-  <xacro:if value="$(arg kinect_enabled)">
-    <xacro:sensor_arch prefix="" parent="top_plate_link">
-      <origin xyz="-0.35 0 0.51" rpy="0 0 -3.14"/>
-    </xacro:sensor_arch>
-    <joint name="kinect_frame_joint" type="fixed">
-      <origin xyz="$(arg kinect_xyz)" rpy="$(arg kinect_rpy)" />
-      <parent link="sensor_arch_mount_link"/>
-      <child link="camera_link"/>
-    </joint>
-    <xacro:kinect_camera prefix="camera" robot_namespace="$(arg robot_namespace)"/>
-  </xacro:if>
   <gazebo>
     <plugin name="gazebo_ros_control" filename="libgazebo_ros_control.so">

File: bramblebee_description/urdf/bramblebee_description.urdf.xacro (robot description, xacro)
@@ -2,7 +2,4 @@
 <!--Software License Agreement (BSD)\file      description.urdf.xacro\authors   Paul Bovbel <pbovbel@clearpathrobotics.com>, Devon Ash <dash@clearpathrobotics.com>\copyright Copyright (c) 2015, Clearpath Robotics, Inc., All rights reserved.Redistribution and use in source and binary forms, with or without modification, are permitted provided thatthe following conditions are met: * Redistributions of source code must retain the above copyright notice, this list of conditions and the   following disclaimer. * Redistributions in binary form must reproduce the above copyright notice, this list of conditions and the   following disclaimer in the documentation and/or other materials provided with the distribution. * Neither the name of Clearpath Robotics nor the names of its contributors may be used to endorse or promote   products derived from this software without specific prior written permission.THIS SOFTWARE IS PROVIDED BY THE COPYRIGHT HOLDERS AND CONTRIBUTORS "AS IS" AND ANY EXPRESS OR IMPLIED WAR-RANTIES, INCLUDING, BUT NOT LIMITED TO, THE IMPLIED WARRANTIES OF MERCHANTABILITY AND FITNESS FOR A PARTICULARPURPOSE ARE DISCLAIMED. IN NO EVENT SHALL THE COPYRIGHT HOLDER OR CONTRIBUTORS BE LIABLE FOR ANY DIRECT, IN-DIRECT, INCIDENTAL, SPECIAL, EXEMPLARY, OR CONSEQUENTIAL DAMAGES (INCLUDING, BUT NOT LIMITED TO, PROCUREMENTOF SUBSTITUTE GOODS OR SERVICES; LOSS OF USE, DATA, OR PROFITS; OR BUSINESS INTERRUPTION) HOWEVER CAUSED ANDON ANY THEORY OF LIABILITY, WHETHER IN CONTRACT, STRICT LIABILITY, OR TORT (INCLUDING NEGLIGENCE OR OTHERWISE)ARISING IN ANY WAY OUT OF THE USE OF THIS SOFTWARE, EVEN IF ADVISED OF THE POSSIBILITY OF SUCH DAMAGE.-->
 <robot name="husky" xmlns:xacro="http://ros.org/wiki/xacro">
-  <xacro:arg name="laser_enabled" default="$(optenv HUSKY_LMS1XX_ENABLED false)" />
-  <xacro:arg name="ur5_enabled" default="$(optenv HUSKY_UR5_ENABLED false)" />
-  <xacro:arg name="kinect_enabled" default="false" />
   <xacro:include filename="$(find bramblebee_description)/urdf/bramblebee.urdf.xacro" />
   <!-- <xacro:husky_robot /> -->
